File: PCB/PCB.kicad_pcb (KiCad board)
At the start: 2 copper layers, 35.6 x 55.9 mm, 40 parts, among them J1 USB_B_Mini, J2 Conn_02x03_Odd_Even, J3 OLED, J4 AudioJack3, Q1 MMBF170, Q2 MMBF170, SW1 SW_Push, SW2 SW_Push, SW3 12CE3xxxxxxTx, SW4 SW_SPST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

Commit message: Updated? pcb files. Modification to CAD. updated gitignore
Parts:
- R11, R12: value R -> 10k
- U1: value ATtiny261A-M -> ATtiny861A-M
