File: PCB/PCB.kicad_sch (KiCad schematic)
At the start: 38 parts, among them J1 USB_B_Mini, J2 Conn_02x03_Odd_Even, J3 OLED, J4 AudioJack3, Q1 MMBF170, Q2 MMBF170, SW1 SW_Push, SW2 SW_Push, SW3 12CE3xxxxxxTx, SW4 SW_SPST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

Commit message: Updated schematic
Parts:
- JP1: value Jumper_2_Open -> (none); footprint Jumper:SolderJumper-2_P1.3mm_Open_RoundedPad1.0x1.5mm -> (none)
Other:
- title: (none) -> Remote Camera Shutter
- moved on the sheet: BT1, C1, C2, C3, C4, C5, D1, F1, H1, H2, J1, J2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

Commit message: Updated? pcb files. Modification to CAD. updated gitignore
Parts:
- removed U1: ATtiny261A-M, Package_DFN_QFN:QFN-32-1EP_5x5mm_P0.5mm_EP3.1x3.1mm, symbol MCU_Microchip_ATtiny:ATtiny261A-M
- added U1: ATtiny861A-M, Package_DFN_QFN:QFN-32-1EP_5x5mm_P0.5mm_EP3.1x3.1mm, symbol MCU_Microchip_ATtiny:ATtiny861A-M
- JP1: value (none) -> Jumper_2_Open; footprint (none) -> Jumper:SolderJumper-2_P1.3mm_Open_RoundedPad1.0x1.5mm
Connections:
- net BT1: now also U1.22 (AREF/PA3)
- net BT2: now also U1.23 (PA2)
- net CHR_STAT: now also U1.10 (PB6)
- net GND: now also U1.21 (AGND), U1.33 (GND), U1.5 (GND)
- net IR_LED: now also U1.15 (PA5)
- net PROG_CLK: now also U1.32 (PB2)
- net PROG_MISO: now also U1.31 (PB1)
- net PROG_MOSI: now also U1.30 (PB0)
- net PROG_RST: now also U1.11 (~{RESET}/PB7)
- net ROTARY_A: now also U1.13 (PA7)
- net ROTARY_B: now also U1.14 (PA6)
- net ROTARY_LED_{B}: now also U1.8 (XTAL2/PB5)
- net ROTARY_LED_{G}: now also U1.2 (PB3)
- net ROTARY_SW: now also U1.7 (XTAL1/PB4)
- net SHUTTER_HOLD: now also U1.25 (PA1)
- net SHUTTER_RELEASE: now also U1.26 (PA0)
- net VCC: now also U1.18 (AVCC), U1.4 (VCC)
- net VCC_SENSE: now also U1.17 (PA4)
